File: pcb/c64sid.kicad_pcb (KiCad board)
At the start: 2 copper layers, 81.4 x 56.2 mm, 16 parts, among them J1 audio_debug, J2 debug, J3 OLED_wit, P1 TRS_JACK, U1 PCF8574A, U2 WeMos_D1_mini, U3 MOS6581, U5 LM386

Commit message: Proef commit
Parts:
- moved J1 4.95 mm to (142.5, 102.3), turned to 90 degrees
- moved J3 2.10 mm to (156.0, 55.2)
- moved J2 1.38 mm to (155.7, 69.7)
- moved R18 1.15 mm to (127.2, 103.3)
Other:
- board text added: "Audio L-R"
- board text added: "D3"
- board text added: "In"
- board text added: "SCL"
- board text added: "SDA"
- board text added: "VCC"
Changed lines of the file:
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@@
   )
   (footprint "Connector_PinHeader_2.54mm:PinHeader_1x03_P2.54mm_Vertical" (layer "F.Cu")
-    (at 144.25 97.67)
+    (at 142.5 102.3 90)
     (descr "Through hole straight pin header, 1x03, 2.54mm pitch, single row")
     (tags "Through hole pin header THT 1x03 2.54mm single row")
@@
     (property "Sheetname" "")
     (attr through_hole)
-    (fp_text reference "J1" (at 0 -2.33) (layer "F.SilkS")
-        (effects (font (size 1 1) (thickness 0.15)))
-    )
-    (fp_text value "audio_debug" (at 0 7.41) (layer "F.Fab")
-        (effects (font (size 1 1) (thickness 0.15)))
-    )
-    (fp_text user "${REFERENCE}" (at 0 2.54 90) (layer "F.Fab")
+    (fp_text reference "J1" (at 0 -2.33 90) (layer "F.SilkS")
+        (effects (font (size 1 1) (thickness 0.15)))
+    )
+    (fp_text value "audio_debug" (at -2.45 2.6 180) (layer "F.Fab")
+        (effects (font (size 1 1) (thickness 0.15)))
+    )
+    (fp_text user "${REFERENCE}" (at 0 2.54) (layer "F.Fab")
         (effects (font (size 1 1) (thickness 0.15)))
     )
@@
     (fp_line (start 1.27 6.35) (end -1.27 6.35)
       (stroke (width 0.1) (type solid)) (layer "F.Fab"))
-    (pad "1" thru_hole rect (at 0 0) (size 1.7 1.7) (drill 1) (layers "*.Cu" "*.Mask")
+    (pad "1" thru_hole rect (at 0 0 90) (size 1.7 1.7) (drill 1) (layers "*.Cu" "*.Mask")
       (net 3 "GND") (pinfunction "Pin_1") (pintype "passive"))
-    (pad "2" thru_hole oval (at 0 2.54) (size 1.7 1.7) (drill 1) (layers "*.Cu" "*.Mask")
+    (pad "2" thru_hole oval (at 0 2.54 90) (size 1.7 1.7) (drill 1) (layers "*.Cu" "*.Mask")
       (net 4 "Audio") (pinfunction "Pin_2") (pintype "passive"))
-    (pad "3" thru_hole oval (at 0 5.08) (size 1.7 1.7) (drill 1) (layers "*.Cu" "*.Mask")
+    (pad "3" thru_hole oval (at 0 5.08 90) (size 1.7 1.7) (drill 1) (layers "*.Cu" "*.Mask")
       (net 4 "Audio") (pinfunction "Pin_3") (pintype "passive"))
     (model "${KICAD6_3DMODEL_DIR}/Connector_PinHeader_2.54mm.3dshapes/PinHeader_1x03_P2.54mm_Vertical.wrl"
@@
   )
   (footprint "Resistor_THT:R_Axial_DIN0204_L3.6mm_D1.6mm_P5.08mm_Horizontal" (layer "F.Cu")
-    (at 127.22 102.2)
+    (at 127.21 103.35)
     (descr "Resistor, Axial_DIN0204 series, Axial, Horizontal, pin pitch=5.08mm, 0.167W, length*diameter=3.6*1.6mm^2, http://cdn-reichelt.de/documents/datenblatt/B400/1_4W%23YAG.pdf")
     (tags "Resistor Axial_DIN0204 series Axial Horizontal pin pitch 5.08mm 0.167W length 3.6mm diameter 1.6mm")
@@
   )
   (footprint "Connector_PinHeader_2.54mm:PinHeader_1x04_P2.54mm_Horizontal" (layer "F.Cu")
-    (at 153.925 55.15)
+    (at 156.025 55.25)
     (descr "Through hole angled pin header, 1x04, 2.54mm pitch, 6mm pin length, single row")
     (tags "Through hole angled pin header THT 1x04 2.54mm single row")
@@
   )
   (footprint "Connector_PinHeader_2.54mm:PinHeader_1x04_P2.54mm_Horizontal" (layer "F.Cu")
-    (at 154.3 69.8)
+    (at 155.675 69.7)
     (descr "Through hole angled pin header, 1x04, 2.54mm pitch, 6mm pin length, single row")
     (tags "Through hole angled pin header THT 1x04 2.54mm single row")
@@
   (gr_line (start 162.9 106.3) (end 167.2 102.1)
     (stroke (width 0.1) (type default)) (layer "Edge.Cuts"))
-  (gr_text "GND" (at 152.3 94 90) (layer "F.SilkS" knockout)
+  (gr_text "GND" (at 152.1 102.25 90) (layer "F.SilkS" knockout)
+    (effects (font (size 0.5 0.5) (thickness 0.125)) (justify left bottom))
+  )
+  (gr_text "SCL" (at 111.3 68.95 90) (layer "F.SilkS")
+    (effects (font (size 0.5 0.5) (thickness 0.125)) (justify left bottom))
+  )
+  (gr_text "SCL" (at 165.6 89.35 90) (layer "F.SilkS")
+    (effects (font (size 0.5 0.5) (thickness 0.125)) (justify left bottom))
+  )
+  (gr_text "VCC" (at 122.9 99.2 90) (layer "F.SilkS")
     (effects (font (size 0.5 0.5) (thickness 0.125)) (justify left bottom))
   )
@@
     (effects (font (size 0.7 0.7) (thickness 0.15)) (justify left bottom))
   )
-  (gr_text "GND" (at 150.55 59.65 90) (layer "F.SilkS" knockout)
+  (gr_text "GND" (at 141.55 100.35) (layer "F.SilkS" knockout)
+    (effects (font (size 0.5 0.5) (thickness 0.125)) (justify left bottom))
+  )
+  (gr_text "GND" (at 153.85 55.95 90) (layer "F.SilkS" knockout)
+    (effects (font (size 0.5 0.5) (thickness 0.125)) (justify left bottom))
+  )
+  (gr_text "D3" (at 153.4 72.8 90) (layer "F.SilkS")
     (effects (font (size 0.5 0.5) (thickness 0.125)) (justify left bottom))
   )
@@
     (effects (font (size 1 1) (thickness 0.15)) (justify left bottom))
   )
-  (gr_text "GND" (at 151.05 78.75 90) (layer "F.SilkS" knockout)
+  (gr_text "GND" (at 153.45 75.4 90) (layer "F.SilkS" knockout)
+    (effects (font (size 0.5 0.5) (thickness 0.125)) (justify left bottom))
+  )
+  (gr_text "SCL" (at 153.85 60.95 90) (layer "F.SilkS")
+    (effects (font (size 0.5 0.5) (thickness 0.125)) (justify left bottom))
+  )
+  (gr_text "VCC" (at 165.55 84.25 90) (layer "F.SilkS")
     (effects (font (size 0.5 0.5) (thickness 0.125)) (justify left bottom))
   )
@@
     (effects (font (size 1 1) (thickness 0.15)) (justify left bottom))
   )
-  (gr_text "LM386" (at 118 98.5) (layer "F.SilkS")
+  (gr_text "LM386" (at 117.85 104) (layer "F.SilkS")
     (effects (font (size 1 1) (thickness 0.15)) (justify left bottom))
   )
@@
     (effects (font (size 1 1) (thickness 0.15)) (justify left bottom))
   )
+  (gr_text "VCC" (at 153.4 78.05 90) (layer "F.SilkS")
+    (effects (font (size 0.5 0.5) (thickness 0.125)) (justify left bottom))
+  )
+  (gr_text "SDA" (at 165.55 86.75 90) (layer "F.SilkS")
+    (effects (font (size 0.5 0.5) (thickness 0.125)) (justify left bottom))
+  )
+  (gr_text "VCC" (at 153.85 58.45 90) (layer "F.SilkS")
+    (effects (font (size 0.5 0.5) (thickness 0.125)) (justify left bottom))
+  )
+  (gr_text "Audio L-R" (at 144.3 100.3) (layer "F.SilkS")
+    (effects (font (size 0.5 0.5) (thickness 0.125)) (justify left bottom))
+  )
+  (gr_text "GND" (at 152.25 89.4 90) (layer "F.SilkS" knockout)
+    (effects (font (size 0.5 0.5) (thickness 0.125)) (justify left bottom))
+  )
   (gr_text "GND" (at 143.705 68.8 90) (layer "F.SilkS" knockout)
     (effects (font (size 0.5 0.5) (thickness 0.125)) (justify left bottom))
   )
-  (gr_text "GND" (at 146.2 76.8 90) (layer "F.SilkS" knockout)
-    (effects (font (size 0.5 0.5) (thickness 0.125)) (justify left bottom))
-  )
-  (gr_text "GND" (at 115.2 94.6 90) (layer "F.SilkS" knockout)
+  (gr_text "GND" (at 114.95 101.9 90) (layer "F.SilkS" knockout)
+    (effects (font (size 0.5 0.5) (thickness 0.125)) (justify left bottom))
+  )
+  (gr_text "GND" (at 115.1 96.75 90) (layer "F.SilkS" knockout)
+    (effects (font (size 0.5 0.5) (thickness 0.125)) (justify left bottom))
+  )
+  (gr_text "SDA" (at 153.95 63.6 90) (layer "F.SilkS")
     (effects (font (size 0.5 0.5) (thickness 0.125)) (justify left bottom))
   )
@@
     (effects (font (size 1 1) (thickness 0.15)) (justify left bottom))
   )
+  (gr_text "In" (at 153.5 70.25 90) (layer "F.SilkS")
+    (effects (font (size 0.5 0.5) (thickness 0.125)) (justify left bottom))
+  )
+  (gr_text "SDA" (at 111.35 71.45 90) (layer "F.SilkS")
+    (effects (font (size 0.5 0.5) (thickness 0.125)) (justify left bottom))
+  )
+  (gr_text "GND" (at 152.25 86.85 90) (layer "F.SilkS" knockout)
+    (effects (font (size 0.5 0.5) (thickness 0.125)) (justify left bottom))
+  )
 )

Commit message: Proef commit
Parts:
- moved P1 1.00 mm to (94.2, 100.8)
Routing:
- net GND: track 0.00 -> 155.7 mm
- net VCC: track 0.00 -> 131.2 mm
- net Audio: track 0.00 -> 130.9 mm
- net /SCL: track 0.00 -> 79.9 mm
- net /D3: track 0.00 -> 79.3 mm
- net Net-(U3-CAP2B): track 0.00 -> 74.2 mm
- net /In: track 0.00 -> 74.0 mm
- net /SDA: track 0.00 -> 74.0 mm
- net Net-(U3-OUT): track 0.00 -> 66.7 mm
- net Net-(C5-Pad1): track 0.00 -> 56.5 mm
- net Net-(C3-Pad1): track 0.00 -> 47.5 mm
- net /D4: track 0.00 -> 44.2 mm
- net /D5: track 0.00 -> 41.5 mm
- net /D6: track 0.00 -> 41.3 mm
- net /D7: track 0.00 -> 41.3 mm
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